File: hardware/microcontroler/microcontroler.kicad_sch (KiCad schematic)
At the start: 11 parts, among them U1 STM32L021K4Tx

Commit message: progress
Parts:
- added C6, C7: 1uF, symbol Device:C_Small
- added C8: 100n, symbol Device:C_Small
- added C9: 10u, symbol Device:C_Small
- added D3: GREEN LED, symbol Device:LED_Small
- added R3: 1k, symbol Device:R_Small
- added U2: BU33SD5WG-TR, Package_TO_SOT_SMD:SOT-23-5, symbol Regulator_Linear:MCP1802x-xx02xOT
- added U3: MCP4801-E/SN, symbol Analog_DAC:MCP4801
Connections:
- net +3.3V: now also C7.1, D3.2 (A), U2.5 (VOUT)
- net +3.3VA: now also C8.1, C9.1, U3.1 (Vdd), U3.6 (~{SHDN})
- net DAC_nCS: now also U3.2 (~{CS})
- net DAC_nLDAC: now also U3.5 (~{LDAC})
- net GND: now also C6.2, C7.2, C8.2, C9.2, R3.2, U2.2 (GND), U3.7 (Vss)
- net SPI1_MOSI: now also U3.4 (SDI)
- net SPI1_SCK: now also U3.3 (SCK)
- new net: D3.1 (K), R3.1
- new net +5V: C6.1, U2.1 (VIN), U2.3 (~{SHDN})
- new net DAC_OUT: U3.8 (Vout)
Other:
- note added: "DAC MCP4801 :)"
- note added: "Power supply :)"
